File: KiCad/onoff_ampli_board/onoff_ampli_board.sch (KiCad schematic (older format))
At the start: 9 parts, among them K101 Finder 40.31, K102 Finder 40.31, P101 CONN_2, P102 CONN_2, P103 CONN_2, P104 CONN_2

Commit message: Correctifs divers
Parts:
- K101, K102: footprint franck:Relay_40.31_Finder -> flem:Relay_40.31_Finder
- P102, P103: footprint franck:CONN_AK350_02_7.62 -> flem:CONN_AK350_02_7.62
Changed lines of the file:
@@
 F 0 "K102" H 7450 4500 60  0000 C CNN
 F 1 "Finder 40.31" H 7450 3900 60  0000 C CNN
-F 2 "franck:Relay_40.31_Finder" H 7450 4100 60  0001 C CNN
+F 2 "flem:Relay_40.31_Finder" H 7450 4100 60  0001 C CNN
 F 3 "" H 7450 4100 60  0000 C CNN
 	1    7450 4100
@@
 F 0 "K101" H 7450 2600 60  0000 C CNN
 F 1 "Finder 40.31" H 7450 2000 60  0000 C CNN
-F 2 "franck:Relay_40.31_Finder" H 7450 2200 60  0001 C CNN
+F 2 "flem:Relay_40.31_Finder" H 7450 2200 60  0001 C CNN
 F 3 "" H 7450 2200 60  0000 C CNN
 	1    7450 2200
@@
 F 0 "P102" V 4500 2900 40  0000 C CNN
 F 1 "CONN_2" V 4600 2900 40  0000 C CNN
-F 2 "franck:CONN_AK350_02_7.62" H 4550 2900 60  0001 C CNN
+F 2 "flem:CONN_AK350_02_7.62" H 4550 2900 60  0001 C CNN
 F 3 "" H 4550 2900 60  0000 C CNN
 	1    4550 2900
@@
 F 0 "P103" V 4500 3450 40  0000 C CNN
 F 1 "CONN_2" V 4600 3450 40  0000 C CNN
-F 2 "franck:CONN_AK350_02_7.62" H 4550 3450 60  0001 C CNN
+F 2 "flem:CONN_AK350_02_7.62" H 4550 3450 60  0001 C CNN
 F 3 "" H 4550 3450 60  0000 C CNN
 	1    4550 3450
