File: KiCad/onoff_ampli_board/onoff_ampli_board.kicad_pcb (KiCad board)
At the start: 2 copper layers, 62.2 x 49.5 mm, 13 parts, among them K101 Finder 40.31, K102 Finder 40.31, P101 CONN_2, P102 CONN_2, P103 CONN_2, P104 CONN_2

Commit message: Correctifs divers
Parts:
- K101, K102: footprint franck:Relay_40.31_Finder -> flem:Relay_40.31_Finder
- P102, P103: footprint franck:CONN_AK350_02_7.62 -> flem:CONN_AK350_02_7.62
Changed lines of the file:
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@@
     )
   )
-  (module franck:Relay_40.31_Finder (layer F.Cu)
+  (module flem:Relay_40.31_Finder (layer F.Cu)
     (at 128.27 83.82)
     (descr "Relay, SPST, Schrack-RP-II/1, RM3.5mm, 8A250VAC")
@@
       (net 4 /P.OUT))
   )
-  (module franck:Relay_40.31_Finder (layer F.Cu)
+  (module flem:Relay_40.31_Finder (layer F.Cu)
     (at 128.27 101.6)
     (descr "Relay, SPST, Schrack-RP-II/1, RM3.5mm, 8A250VAC")
@@
       (net 6 /N.OUT))
   )
-  (module franck:CONN_AK350_02_7.62 (layer F.Cu)
+  (module flem:CONN_AK350_02_7.62 (layer F.Cu)
     (at 153.67 114.3)
     (attr virtual)
-    (fp_text reference P102 (at 3.81 -3.81) (layer F.SilkS)
+    (fp_text reference P102 (at 3.81 -8.255) (layer F.SilkS)
       (effects (font (size 1 1) (thickness 0.15)))
     )
-    (fp_text value CONN_2 (at 3.81 6.35) (layer F.SilkS)
+    (fp_text value CONN_2 (at 3.81 2.54) (layer F.SilkS)
       (effects (font (size 1 1) (thickness 0.15)))
     )
@@
       (net 3 /P.IN))
   )
-  (module franck:CONN_AK350_02_7.62 (layer F.Cu)
+  (module flem:CONN_AK350_02_7.62 (layer F.Cu)
     (at 138.43 114.3)
     (attr virtual)
-    (fp_text reference P103 (at 3.81 -3.81) (layer F.SilkS)
+    (fp_text reference P103 (at 3.81 -8.255) (layer F.SilkS)
       (effects (font (size 1 1) (thickness 0.15)))
     )
-    (fp_text value CONN_2 (at 3.81 6.35) (layer F.SilkS)
+    (fp_text value CONN_2 (at 3.81 2.54) (layer F.SilkS)
       (effects (font (size 1 1) (thickness 0.15)))
     )

Commit message: Gerber
Parts:
- moved REF** 1.27 mm to (171.4, 74.9)
- moved REF** 1.27 mm to (171.4, 116.8)
Other:
- board size 62.2 x 49.5 mm -> 63.5 x 49.5 mm
Changed lines of the file:
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@@
     (links 16)
     (no_connects 0)
-    (area 104.227143 69.755 184.403334 127.730001)
+    (area 104.227143 69.755 186.943334 129.000001)
     (thickness 1.6)
     (drawings 10)
@@
     (mod_text_size 1 1)
     (mod_text_width 0.15)
-    (pad_size 1 1)
-    (pad_drill 0.6)
+    (pad_size 3 3)
+    (pad_drill 1.6)
     (pad_to_mask_clearance 0.1)
     (aux_axis_origin 138.43 114.3)
@@
     (fp_line (start 27.94 2.54) (end -2.54 2.54) (layer F.SilkS) (width 0.381))
     (fp_line (start -2.54 2.54) (end -2.54 -10.16) (layer F.SilkS) (width 0.381))
-    (pad 12 thru_hole circle (at 16.51 0) (size 3.6 3.6) (drill 1.6) (layers *.Cu *.Mask F.SilkS))
+    (pad 12 thru_hole circle (at 16.51 0) (size 3 3) (drill 1.6) (layers *.Cu *.Mask F.SilkS))
     (pad A2 thru_hole circle (at 0 -7.62) (size 3.4 3.4) (drill 1.6) (layers *.Cu *.Mask F.SilkS)
       (net 1 /K))
@@
     (fp_line (start 27.94 2.54) (end -2.54 2.54) (layer F.SilkS) (width 0.381))
     (fp_line (start -2.54 2.54) (end -2.54 -10.16) (layer F.SilkS) (width 0.381))
-    (pad 12 thru_hole circle (at 16.51 0) (size 3.6 3.6) (drill 1.6) (layers *.Cu *.Mask F.SilkS))
+    (pad 12 thru_hole circle (at 16.51 0) (size 3 3) (drill 1.6) (layers *.Cu *.Mask F.SilkS))
     (pad A2 thru_hole circle (at 0 -7.62) (size 3.4 3.4) (drill 1.6) (layers *.Cu *.Mask F.SilkS)
       (net 1 /K))
@@
   )
   (module Mounting_Holes:MountingHole_3.2mm_M3_Pad (layer F.Cu)
-    (at 170.18 74.93)
+    (at 171.45 74.93)
     (descr "Mounting Hole 3.2mm, M3")
     (tags "mounting hole 3.2mm m3")
@@
   )
   (module Mounting_Holes:MountingHole_3.2mm_M3_Pad (layer F.Cu)
-    (at 170.18 116.84)
+    (at 171.45 116.84)
     (descr "Mounting Hole 3.2mm, M3")
     (tags "mounting hole 3.2mm m3")
@@
   )
   (dimension 49.53 (width 0.25) (layer Cmts.User)
-    (gr_text "49,530 mm" (at 180.07 95.885 270) (layer Cmts.User)
+    (gr_text "49,530 mm" (at 182.61 95.885 270) (layer Cmts.User)
       (effects (font (size 1 1) (thickness 0.25)))
     )
-    (feature1 (pts (xy 173.99 120.65) (xy 181.07 120.65)))
-    (feature2 (pts (xy 173.99 71.12) (xy 181.07 71.12)))
-    (crossbar (pts (xy 179.07 71.12) (xy 179.07 120.65)))
-    (arrow1a (pts (xy 179.07 120.65) (xy 178.483579 119.523496)))
-    (arrow1b (pts (xy 179.07 120.65) (xy 179.656421 119.523496)))
-    (arrow2a (pts (xy 179.07 71.12) (xy 178.483579 72.246504)))
-    (arrow2b (pts (xy 179.07 71.12) (xy 179.656421 72.246504)))
-  )
-  (dimension 62.23 (width 0.25) (layer Cmts.User)
-    (gr_text "62,230 mm" (at 142.875 126.73) (layer Cmts.User)
+    (feature1 (pts (xy 175.26 120.65) (xy 183.61 120.65)))
+    (feature2 (pts (xy 175.26 71.12) (xy 183.61 71.12)))
+    (crossbar (pts (xy 181.61 71.12) (xy 181.61 120.65)))
+    (arrow1a (pts (xy 181.61 120.65) (xy 181.023579 119.523496)))
+    (arrow1b (pts (xy 181.61 120.65) (xy 182.196421 119.523496)))
+    (arrow2a (pts (xy 181.61 71.12) (xy 181.023579 72.246504)))
+    (arrow2b (pts (xy 181.61 71.12) (xy 182.196421 72.246504)))
+  )
+  (dimension 63.5 (width 0.25) (layer Cmts.User)
+    (gr_text "63,500 mm" (at 143.51 128) (layer Cmts.User)
       (effects (font (size 1 1) (thickness 0.25)))
     )
-    (feature1 (pts (xy 173.99 120.65) (xy 173.99 127.73)))
-    (feature2 (pts (xy 111.76 120.65) (xy 111.76 127.73)))
-    (crossbar (pts (xy 111.76 125.73) (xy 173.99 125.73)))
-    (arrow1a (pts (xy 173.99 125.73) (xy 172.863496 126.316421)))
-    (arrow1b (pts (xy 173.99 125.73) (xy 172.863496 125.143579)))
-    (arrow2a (pts (xy 111.76 125.73) (xy 112.886504 126.316421)))
-    (arrow2b (pts (xy 111.76 125.73) (xy 112.886504 125.143579)))
-  )
+    (feature1 (pts (xy 175.26 120.65) (xy 175.26 129)))
+    (feature2 (pts (xy 111.76 120.65) (xy 111.76 129)))
+    (crossbar (pts (xy 111.76 127) (xy 175.26 127)))
+    (arrow1a (pts (xy 175.26 127) (xy 174.133496 127.586421)))
+    (arrow1b (pts (xy 175.26 127) (xy 174.133496 126.413579)))
+    (arrow2a (pts (xy 111.76 127) (xy 112.886504 127.586421)))
+    (arrow2b (pts (xy 111.76 127) (xy 112.886504 126.413579)))
+  )
+  (gr_line (start 175.26 71.12) (end 175.26 120.65) (angle 90) (layer Edge.Cuts) (width 0.15))
   (gr_text N.OUT (at 146.05 107.95) (layer F.SilkS)
     (effects (font (size 1 1) (thickness 0.25)))
@@
   )
   (gr_line (start 111.76 120.65) (end 111.76 71.12) (angle 90) (layer Edge.Cuts) (width 0.15))
-  (gr_line (start 173.99 120.65) (end 111.76 120.65) (angle 90) (layer Edge.Cuts) (width 0.15))
-  (gr_line (start 173.99 71.12) (end 173.99 120.65) (angle 90) (layer Edge.Cuts) (width 0.15))
-  (gr_line (start 111.76 71.12) (end 173.99 71.12) (angle 90) (layer Edge.Cuts) (width 0.15))
+  (gr_line (start 175.26 120.65) (end 111.76 120.65) (angle 90) (layer Edge.Cuts) (width 0.15))
+  (gr_line (start 111.76 71.12) (end 175.26 71.12) (angle 90) (layer Edge.Cuts) (width 0.15))
   (segment (start 123.19 92.71) (end 116.84 99.06) (width 0.381) (layer F.Cu) (net 1))
   (segment (start 116.84 99.06) (end 116.84 100.33) (width 0.381) (layer F.Cu) (net 1))
