File: KiCad/power_board/power_board.sch (KiCad schematic (older format))
At the start: 51 parts, among them K101 DS-BT, P101 CONN_01X03, P102 CONN_01X03, P103 CONN_01X03, P104 CONN_02X04, P105 CONN_02X02, P106 CONN_02X02, P107 CONN_02X03, P108 CONN_01X06, U101 HLK-PM01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

Commit message: Correctifs divers
Parts:
- D105: footprint franck:Bridge -> flem:Bridge
- K101: footprint franck:Relay_DS-BT_Nais -> flem:Relay_DS-BT_Nais
- P101, P102, P103: footprint franck:CONN_AK350_03_5.08 -> flem:CONN_AK350_03_5.08
- U101: footprint franck:HLK-PM01 -> flem:HLK-PM01
Changed lines of the file:
@@
 F 0 "K101" H 7300 1600 70  0000 C CNN
 F 1 "DS-BT" H 7350 700 70  0000 C CNN
-F 2 "franck:Relay_DS-BT_Nais" H 7350 1200 60  0001 C CNN
+F 2 "flem:Relay_DS-BT_Nais" H 7350 1200 60  0001 C CNN
 F 3 "" H 7350 1200 60  0000 C CNN
 	1    7350 1200
@@
 F 0 "U101" H 2300 1450 60  0000 C CNN
 F 1 "HLK-PM01" H 2300 1150 60  0000 C CNN
-F 2 "franck:HLK-PM01" H 2300 1150 60  0001 C CNN
+F 2 "flem:HLK-PM01" H 2300 1150 60  0001 C CNN
 F 3 "" H 2300 1150 60  0000 C CNN
 	1    2300 1150
@@
 F 0 "P101" H 900 2100 50  0000 C CNN
 F 1 "CONN_01X03" V 1050 1900 50  0000 C CNN
-F 2 "franck:CONN_AK350_03_5.08" H 950 1900 50  0001 C CNN
+F 2 "flem:CONN_AK350_03_5.08" H 950 1900 50  0001 C CNN
 F 3 "" H 950 1900 50  0000 C CNN
 	1    950  1900
@@
 F 0 "P103" H 9300 1350 50  0000 C CNN
 F 1 "CONN_01X03" V 9400 1150 50  0000 C CNN
-F 2 "franck:CONN_AK350_03_5.08" H 9300 1150 50  0001 C CNN
+F 2 "flem:CONN_AK350_03_5.08" H 9300 1150 50  0001 C CNN
 F 3 "" H 9300 1150 50  0000 C CNN
 	1    9300 1150
@@
 F 0 "P102" H 2150 3300 50  0000 C CNN
 F 1 "CONN_01X03" V 2300 3100 50  0000 C CNN
-F 2 "franck:CONN_AK350_03_5.08" H 2200 3100 50  0001 C CNN
+F 2 "flem:CONN_AK350_03_5.08" H 2200 3100 50  0001 C CNN
 F 3 "" H 2200 3100 50  0000 C CNN
 	1    2200 3100
@@
 F 0 "D105" H 4100 3575 50  0000 L CNN
 F 1 "D_Bridge_-A+A" H 4100 3500 50  0000 L CNN
-F 2 "franck:Bridge" H 4050 3300 50  0001 C CNN
+F 2 "flem:Bridge" H 4050 3300 50  0001 C CNN
 F 3 "" H 4050 3300 50  0001 C CNN
 	1    4050 3300
