File: KiCad/power_board/power_board.kicad_pcb (KiCad board)
At the start: 2 copper layers, 99.1 x 86.4 mm, 56 parts, among them K101 DS-BT, P101 CONN_01X03, P102 CONN_01X03, P103 CONN_01X03, P104 CONN_02X04, P105 CONN_02X02, P106 CONN_02X02, P107 CONN_02X03, P108 CONN_01X06, U101 HLK-PM01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

Commit message: Correctifs divers
Parts:
- D105: footprint franck:Bridge -> flem:Bridge
- K101: footprint franck:Relay_DS-BT_Nais -> flem:Relay_DS-BT_Nais
- P101, P102, P103: footprint franck:CONN_AK350_03_5.08 -> flem:CONN_AK350_03_5.08
- U101: footprint franck:HLK-PM01 -> flem:HLK-PM01
Changed lines of the file:
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@@
     (links 110)
     (no_connects 0)
-    (area 54.356667 36.1 171.362858 129.735)
+    (area 65.964999 43.104999 165.175001 129.615001)
     (thickness 1.6)
     (drawings 6)
@@
     (add_net "Net-(D104-Pad2)")
   )
-  (module franck:CONN_AK350_03_5.08 (layer F.Cu)
+  (module flem:CONN_AK350_03_5.08 (layer F.Cu)
     (at 134.62 49.53 180)
     (attr virtual)
@@
     )
   )
-  (module franck:HLK-PM01 (layer F.Cu)
+  (module flem:HLK-PM01 (layer F.Cu)
     (at 77.47 74.295 270)
     (fp_text reference U101 (at -0.635 -11.43 270) (layer F.SilkS)
@@
     )
   )
-  (module franck:CONN_AK350_03_5.08 (layer F.Cu)
+  (module flem:CONN_AK350_03_5.08 (layer F.Cu)
     (at 91.44 49.53 180)
     (attr virtual)
@@
       (net 19 /Phase))
   )
-  (module franck:CONN_AK350_03_5.08 (layer F.Cu)
+  (module flem:CONN_AK350_03_5.08 (layer F.Cu)
     (at 106.68 49.53 180)
     (attr virtual)
@@
       (net 22 /Torique_0_Blue))
   )
-  (module franck:Relay_DS-BT_Nais (layer F.Cu)
+  (module flem:Relay_DS-BT_Nais (layer F.Cu)
     (at 91.44 68.58)
     (descr "Relay, DS-BT, Nais")
@@
     )
   )
-  (module franck:Bridge (layer F.Cu)
+  (module flem:Bridge (layer F.Cu)
     (at 128.27 59.69 180)
     (descr "Support fusible 5 x 20")

Commit message: Gerber
Parts:
- moved REF** 1.27 mm to (69.8, 48.3)
- moved REF** 1.27 mm to (69.8, 124.5)
- moved REF** 1.27 mm to (113.0, 120.7)
- moved REF** 1.27 mm to (161.3, 48.3)
- moved REF** 1.27 mm to (161.3, 124.5)
Other:
- board size 99.1 x 86.4 mm -> 99.1 x 83.8 mm
Changed lines of the file:
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@@
     (links 110)
     (no_connects 0)
-    (area 65.964999 43.104999 165.175001 129.615001)
+    (area 54.356667 36.1 172.632858 129.735)
     (thickness 1.6)
     (drawings 6)
@@
   )
   (module Mounting_Holes:MountingHole_3.2mm_M3_Pad (layer F.Cu)
-    (at 71.12 48.26)
+    (at 69.85 48.26)
     (descr "Mounting Hole 3.2mm, M3")
     (tags "mounting hole 3.2mm m3")
@@
   )
   (module Mounting_Holes:MountingHole_3.2mm_M3_Pad (layer F.Cu)
-    (at 114.3 120.65)
+    (at 113.03 120.65)
     (descr "Mounting Hole 3.2mm, M3")
     (tags "mounting hole 3.2mm m3")
@@
   )
   (module Mounting_Holes:MountingHole_3.2mm_M3_Pad (layer F.Cu)
-    (at 160.02 48.26)
+    (at 161.29 48.26)
     (descr "Mounting Hole 3.2mm, M3")
     (tags "mounting hole 3.2mm m3")
@@
   )
   (module Mounting_Holes:MountingHole_3.2mm_M3_Pad (layer F.Cu)
-    (at 71.12 124.46)
+    (at 69.85 124.46)
     (descr "Mounting Hole 3.2mm, M3")
     (tags "mounting hole 3.2mm m3")
@@
   )
   (module Mounting_Holes:MountingHole_3.2mm_M3_Pad (layer F.Cu)
-    (at 160.02 124.46)
+    (at 161.29 124.46)
     (descr "Mounting Hole 3.2mm, M3")
     (tags "mounting hole 3.2mm m3")
@@
     (pad 1 thru_hole circle (at 0 0) (size 6.4 6.4) (drill 3.2) (layers *.Cu *.Mask))
   )
-  (dimension 86.36 (width 0.25) (layer Cmts.User)
-    (gr_text "86,360 mm" (at 58.69 86.36 270) (layer Cmts.User)
+  (dimension 83.82 (width 0.25) (layer Cmts.User)
+    (gr_text "83,820 mm" (at 58.69 86.36 270) (layer Cmts.User)
       (effects (font (size 1 1) (thickness 0.25)))
     )
-    (feature1 (pts (xy 66.04 129.54) (xy 57.69 129.54)))
-    (feature2 (pts (xy 66.04 43.18) (xy 57.69 43.18)))
-    (crossbar (pts (xy 59.69 43.18) (xy 59.69 129.54)))
-    (arrow1a (pts (xy 59.69 129.54) (xy 59.103579 128.413496)))
-    (arrow1b (pts (xy 59.69 129.54) (xy 60.276421 128.413496)))
-    (arrow2a (pts (xy 59.69 43.18) (xy 59.103579 44.306504)))
-    (arrow2b (pts (xy 59.69 43.18) (xy 60.276421 44.306504)))
+    (feature1 (pts (xy 66.04 128.27) (xy 57.69 128.27)))
+    (feature2 (pts (xy 66.04 44.45) (xy 57.69 44.45)))
+    (crossbar (pts (xy 59.69 44.45) (xy 59.69 128.27)))
+    (arrow1a (pts (xy 59.69 128.27) (xy 59.103579 127.143496)))
+    (arrow1b (pts (xy 59.69 128.27) (xy 60.276421 127.143496)))
+    (arrow2a (pts (xy 59.69 44.45) (xy 59.103579 45.576504)))
+    (arrow2b (pts (xy 59.69 44.45) (xy 60.276421 45.576504)))
   )
   (dimension 99.06 (width 0.25) (layer Cmts.User)
@@
     (arrow2b (pts (xy 66.04 38.1) (xy 67.166504 37.513579)))
   )
-  (gr_line (start 165.1 43.18) (end 165.1 129.54) (angle 90) (layer Edge.Cuts) (width 0.15))
-  (gr_line (start 66.04 43.18) (end 66.04 129.54) (angle 90) (layer Edge.Cuts) (width 0.15))
-  (gr_line (start 165.1 129.54) (end 66.04 129.54) (angle 90) (layer Edge.Cuts) (width 0.15))
-  (gr_line (start 66.04 43.18) (end 165.1 43.18) (angle 90) (layer Edge.Cuts) (width 0.15))
+  (gr_line (start 165.1 44.45) (end 165.1 128.27) (angle 90) (layer Edge.Cuts) (width 0.15))
+  (gr_line (start 66.04 44.45) (end 66.04 128.27) (angle 90) (layer Edge.Cuts) (width 0.15))
+  (gr_line (start 165.1 128.27) (end 66.04 128.27) (angle 90) (layer Edge.Cuts) (width 0.15))
+  (gr_line (start 66.04 44.45) (end 165.1 44.45) (angle 90) (layer Edge.Cuts) (width 0.15))
   (segment (start 151.765 66.04) (end 151.765 74.93) (width 0.508) (layer F.Cu) (net 1))
   (segment (start 141.235 81.915) (end 139.09 84.06) (width 0.508) (layer F.Cu) (net 1))
@@
     (polygon
       (pts
-        (xy 165.1 43.18) (xy 118.11 43.18) (xy 118.11 69.85) (xy 115.57 72.39) (xy 111.76 72.39)
-        (xy 109.22 74.93) (xy 100.33 74.93) (xy 96.52 78.74) (xy 66.04 78.74) (xy 66.04 129.54)
-        (xy 165.1 129.54)
+        (xy 165.1 44.45) (xy 118.11 44.45) (xy 118.11 69.85) (xy 115.57 72.39) (xy 111.76 72.39)
+        (xy 109.22 74.93) (xy 100.33 74.93) (xy 96.52 78.74) (xy 66.04 78.74) (xy 66.04 128.27)
+        (xy 165.1 128.27)
       )
     )
@@
     (polygon
       (pts
-        (xy 165.1 129.54) (xy 165.1 43.18) (xy 118.11 43.18) (xy 118.11 69.85) (xy 115.57 72.39)
+        (xy 165.1 128.27) (xy 165.1 44.45) (xy 118.11 44.45) (xy 118.11 69.85) (xy 115.57 72.39)
         (xy 111.76 72.39) (xy 109.22 74.93) (xy 100.33 74.93) (xy 96.52 78.74) (xy 66.04 78.74)
-        (xy 66.04 129.54)
+        (xy 66.04 128.27)
       )
     )

Commit message: Divers
Changed lines of the file:
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@@
   (segment (start 156.21 72.39) (end 158.75 72.39) (width 0.508) (layer F.Cu) (net 2))
   (segment (start 158.75 72.39) (end 158.75 71.12) (width 0.762) (layer F.Cu) (net 2))
-  (segment (start 93.98 86.68) (end 98.425 91.125) (width 0.508) (layer F.Cu) (net 2))
-  (segment (start 98.425 91.125) (end 98.425 125.095) (width 0.508) (layer F.Cu) (net 2))
+  (segment (start 93.98 86.68) (end 99.06 91.76) (width 0.508) (layer F.Cu) (net 2) (status 400000))
+  (segment (start 99.06 91.76) (end 99.06 125.095) (width 0.508) (layer F.Cu) (net 2))
   (segment (start 114.3 83.82) (end 114.3 85.09) (width 0.508) (layer B.Cu) (net 2))
   (segment (start 73.04 85.725) (end 69.77 88.995) (width 0.508) (layer B.Cu) (net 2))
@@
   (segment (start 142.24 95.25) (end 143.51 93.98) (width 0.508) (layer B.Cu) (net 4))
   (segment (start 158.75 82.55) (end 158.75 83.82) (width 0.762) (layer B.Cu) (net 4))
-  (segment (start 156.845 82.55) (end 158.75 82.55) (width 0.508) (layer B.Cu) (net 4))
-  (segment (start 145.415 93.98) (end 156.845 82.55) (width 0.508) (layer B.Cu) (net 4))
-  (segment (start 143.51 93.98) (end 145.415 93.98) (width 0.508) (layer B.Cu) (net 4))
+  (segment (start 154.94 82.55) (end 158.75 82.55) (width 0.508) (layer B.Cu) (net 4))
+  (segment (start 143.51 93.98) (end 154.94 82.55) (width 0.508) (layer B.Cu) (net 4))
+  (segment (start 143.51 93.98) (end 143.51 93.98) (width 0.508) (layer B.Cu) (net 4))
   (segment (start 130.81 88.9) (end 130.81 71.12) (width 0.508) (layer F.Cu) (net 4))
   (segment (start 140.335 50.705) (end 142.24 48.8) (width 0.508) (layer F.Cu) (net 4))
@@
   (segment (start 93.98 122.555) (end 93.98 124.46) (width 0.508) (layer B.Cu) (net 5))
   (segment (start 98.425 118.11) (end 93.98 122.555) (width 0.508) (layer B.Cu) (net 5))
-  (segment (start 100.965 118.11) (end 98.425 118.11) (width 0.508) (layer B.Cu) (net 5))
-  (via (at 100.965 118.11) (size 0.6) (drill 0.4) (layers F.Cu B.Cu) (net 5))
-  (segment (start 100.965 95.885) (end 100.965 118.11) (width 0.508) (layer F.Cu) (net 5))
-  (segment (start 108.585 88.265) (end 100.965 95.885) (width 0.508) (layer F.Cu) (net 5))
+  (segment (start 101.6 118.11) (end 98.425 118.11) (width 0.508) (layer B.Cu) (net 5))
+  (via (at 101.6 118.11) (size 0.6) (drill 0.4) (layers F.Cu B.Cu) (net 5))
+  (segment (start 101.6 95.25) (end 101.6 118.11) (width 0.508) (layer F.Cu) (net 5))
+  (segment (start 108.585 88.265) (end 101.6 95.25) (width 0.508) (layer F.Cu) (net 5))
   (segment (start 108.585 84.455) (end 108.585 88.265) (width 0.508) (layer F.Cu) (net 5))
   (segment (start 153.67 88.9) (end 153.67 76.835) (width 0.508) (layer F.Cu) (net 6))
@@
   (segment (start 133.35 86.995) (end 133.985 86.36) (width 0.508) (layer F.Cu) (net 6))
   (segment (start 133.985 86.36) (end 139.09 86.36) (width 0.508) (layer F.Cu) (net 6))
-  (segment (start 102.87 83.82) (end 99.695 86.995) (width 0.508) (layer F.Cu) (net 6))
+  (segment (start 102.87 83.82) (end 100.33 86.36) (width 0.508) (layer F.Cu) (net 6) (status 400000))
   (segment (start 96.52 122.555) (end 96.52 124.46) (width 0.508) (layer B.Cu) (net 6))
   (segment (start 98.425 120.65) (end 96.52 122.555) (width 0.508) (layer B.Cu) (net 6))
-  (segment (start 99.695 120.65) (end 98.425 120.65) (width 0.508) (layer B.Cu) (net 6))
-  (via (at 99.695 120.65) (size 0.6) (drill 0.4) (layers F.Cu B.Cu) (net 6))
-  (segment (start 99.695 86.995) (end 99.695 120.65) (width 0.508) (layer F.Cu) (net 6))
+  (segment (start 100.33 120.65) (end 98.425 120.65) (width 0.508) (layer B.Cu) (net 6))
+  (via (at 100.33 120.65) (size 0.6) (drill 0.4) (layers F.Cu B.Cu) (net 6))
+  (segment (start 100.33 86.36) (end 100.33 120.65) (width 0.508) (layer F.Cu) (net 6))
   (segment (start 158.75 86.36) (end 161.29 86.36) (width 0.762) (layer B.Cu) (net 6))
   (segment (start 161.29 86.36) (end 161.29 88.9) (width 0.762) (layer B.Cu) (net 6))
@@
   (segment (start 120.015 85.09) (end 114.935 80.01) (width 0.508) (layer F.Cu) (net 25))
   (segment (start 120.015 98.425) (end 120.015 85.09) (width 0.508) (layer F.Cu) (net 25))
-  (segment (start 152.4 102.87) (end 145.415 102.87) (width 0.508) (layer B.Cu) (net 25))
+  (segment (start 152.4 102.87) (end 152.4 102.87) (width 0.508) (layer B.Cu) (net 25) (status C00000))
   (segment (start 131.445 102.87) (end 124.46 102.87) (width 0.508) (layer B.Cu) (net 25))
   (segment (start 133.985 100.33) (end 131.445 102.87) (width 0.508) (layer B.Cu) (net 25))
-  (segment (start 142.875 100.33) (end 133.985 100.33) (width 0.508) (layer B.Cu) (net 25))
-  (segment (start 145.415 102.87) (end 142.875 100.33) (width 0.508) (layer B.Cu) (net 25))
+  (segment (start 149.86 100.33) (end 133.985 100.33) (width 0.508) (layer B.Cu) (net 25))
+  (segment (start 152.4 102.87) (end 149.86 100.33) (width 0.508) (layer B.Cu) (net 25) (status 400000))
   (segment (start 148.59 118.11) (end 148.59 113.03) (width 0.508) (layer F.Cu) (net 25))
   (segment (start 151.67 109.95) (end 151.67 107.95) (width 0.508) (layer F.Cu) (net 25))
