File: KiCad/ampli_hifi/ampli_hifi.sch (KiCad schematic (older format))
At the start: 8 parts, among them T101 Torique 2x9v

Commit message: Divers
Parts:
- removed U?: APA-106, symbol APA-106
Connections:
- net MCU Board 587ABF07/LED_PWR_A: now also D?.2 (A)
- net MCU Board 587ABF07/LED_PWR_K: now also D?.1 (K)
- no-connect marks 1 -> 0
Changed lines of the file:
@@
 EESchema Schematic File Version 2
+LIBS:ampli_hifi-rescue
 LIBS:power
 LIBS:device
@@
 $Descr A3 16535 11693
 encoding utf-8
-Sheet 1 6
+Sheet 1 7
 Title "Préamplificateur HiFi"
 Date "2017-01-14"
@@
 $EndComp
 Wire Wire Line
-	4100 5400 4550 5400
-Wire Wire Line
-	4950 5400 4950 5400
+	4100 5400 4600 5400
+Wire Wire Line
+	4900 5400 4950 5400
 Wire Wire Line
 	4950 5400 4950 5500
 Wire Wire Line
 	4950 5500 4100 5500
-$Comp
-L APA-106 U?
-U 1 1 58886548
-P 4900 5950
-F 0 "U?" H 4700 6250 60  0000 C CNN
-F 1 "APA-106" H 4900 5650 60  0000 C CNN
-F 2 "" H 4900 5500 60  0000 C CNN
-F 3 "" H 4900 5500 60  0000 C CNN
-	1    4900 5950
-	1    0    0    -1
-$EndComp
 $Comp
 L +5P #PWR?
@@
 Wire Wire Line
 	1950 2650 2300 2650
-$Comp
-L GND #PWR?
-U 1 1 5888CEC9
-P 5400 6100
-F 0 "#PWR?" H 5400 5850 50  0001 C CNN
-F 1 "GND" H 5400 5950 50  0000 C CNN
-F 2 "" H 5400 6100 50  0000 C CNN
-F 3 "" H 5400 6100 50  0000 C CNN
-	1    5400 6100
-	0    -1   -1   0
-$EndComp
-Wire Wire Line
-	5350 6100 5400 6100
-NoConn ~ 5350 5800
 $Sheet
 S 2300 6200 1800 2200

Commit message: Divers
Parts:
- removed D?: LED, symbol LED
- removed J?: DB9, symbol DB9
- added U?: NEOPIXEL, symbol NEOPIXEL
Connections:
- net +5P: now also U?.2 (VDD)
- net MCU Board 587ABF07/Neutre renamed Power Board Sheet588FD2C2/Neutre
- net MCU Board 587ABF07/Phase renamed Power Board Sheet588FD2C2/Phase
- net MCU Board 587ABF07/Terre renamed Power Board Sheet588FD2C2/Terre
- net MCU Board 587ABF07/Torique_0_Black_9_Yellow renamed Power Board Sheet588FD2C2/Torique_0_Black_9_Yellow
- net MCU Board 587ABF07/Torique_0_Blue renamed Power Board Sheet588FD2C2/Torique_0_Blue
- net MCU Board 587ABF07/Torique_0_Orange renamed Power Board Sheet588FD2C2/Torique_0_Orange
- net MCU Board 587ABF07/Torique_0_Violet renamed Power Board Sheet588FD2C2/Torique_0_Violet
- net MCU Board 587ABF07/Torique_115_Brown renamed Power Board Sheet588FD2C2/Torique_115_Brown
- net MCU Board 587ABF07/Torique_115_Grey renamed Power Board Sheet588FD2C2/Torique_115_Grey
- net MCU Board 587ABF07/Torique_9_Red renamed Power Board Sheet588FD2C2/Torique_9_Red
- new net MCU Board 587ABF07/LED_DIN: U?.1 (DIN)
- new net MCU Board 587ABF07/LED_GND: U?.3 (GND)
- no-connect marks 0 -> 1
Other:
- moved on the sheet: DS101, Neutre101, Phase101, T101, Terre101
