File: KiCad/select_board/select_board.sch (KiCad schematic (older format))
At the start: 67 parts, among them J101 RCA, J102 RCA, J103 RCA, J104 RCA, J105 TAPE_OUT_L, J106 TAPE_OUT_R, J107 RCA, J108 RCA, J109 RCA, J110 RCA, J111 RCA, J112 RCA, J113 RCA, J114 RCA, J115 RCA, J116 RCA, J117 PRE_OUT_L, J118 PRE_OUT_R, K101 TQ2, K102 TQ2, K103 TQ2, K104 TQ2, K105 TQ2, K106 TQ2, K107 TQ2, K108 TQ2, P101 CONN_1, P102 CONN_1, P103 CONN_1, P104 CONN_1, P105 CONN_01X10

Commit message: PCB select_board
Parts:
- removed D107, D108: 1N4148, Discret:DO-35, symbol D
- removed J105: TAPE_OUT_L, symbol RCA
- removed J106: TAPE_OUT_R, symbol RCA
- removed J113, J115, J116: RCA, symbol RCA
- removed K101, K102, K103, K104, K105, K106, K107, K108: TQ2, flem:Relay_TQ2_Nais, symbol TQ2_ABC
- removed P105: CONN_01X10, symbol CONN_01X10
- removed PA101, PA102, PB101, PB102: CONN_1, symbol CONN_1
- removed PC101: PHONE_L, symbol CONN_1
- removed PC102: PHONE_R, symbol CONN_1
- removed PD101: PHONE_L_GND, symbol CONN_1
- removed PD102: PHONE_R_GND, symbol CONN_1
- removed R103, R104: 470, Resistors_ThroughHole:Resistor_Horizontal_RM10mm, symbol R
- removed R113, R114, R115, R116: 47K, Resistors_ThroughHole:Resistor_Horizontal_RM10mm, symbol R
- added J112: BY_PASS_L, flem:RCA_ELECAUDIO_ER107, symbol RCA
- added K101, K102, K103, K104, K105, K106: G6K, flem:Omron-G6K-2F-Y, symbol Omron-G6K-2F-Y_ABC
- added P105: CONN_01X07, Pin_Headers:Pin_Header_Straight_1x07_Pitch2.54mm, symbol CONN_01X07
- D101, D102, D103, D104, D105, D106: footprint Discret:DO-35 -> Diodes_ThroughHole:D_DO-35_SOD27_P7.62mm_Horizontal
- J101, J102, J103, J104: footprint (none) -> flem:RCA_ELECAUDIO_ER107
- J105: renamed from J107; footprint (none) -> flem:RCA_ELECAUDIO_ER107
- J106: renamed from J108; footprint (none) -> flem:RCA_ELECAUDIO_ER107
- J107: renamed from J109; footprint (none) -> flem:RCA_ELECAUDIO_ER107
- J108: renamed from J110; footprint (none) -> flem:RCA_ELECAUDIO_ER107
- J109: renamed from J111; footprint (none) -> flem:RCA_ELECAUDIO_ER107
- J110: renamed from J112; footprint (none) -> flem:RCA_ELECAUDIO_ER107
- J111: renamed from J117; footprint (none) -> flem:RCA_ELECAUDIO_ER107
- J113: renamed from J118; footprint (none) -> flem:RCA_ELECAUDIO_ER107
- J114: value RCA -> BY_PASS_R; footprint (none) -> flem:RCA_ELECAUDIO_ER107
- PA101: renamed from P101; footprint (none) -> flem:1Pin_d1.8mm_D3.4mm
- PA102: renamed from P103; footprint (none) -> flem:1Pin_d1.8mm_D3.4mm
- PA103, PA104, PB103, PB104: footprint (none) -> flem:1Pin_d1.8mm_D3.4mm
- PB101: renamed from P102; footprint (none) -> flem:1Pin_d1.8mm_D3.4mm
- PB102: renamed from P104; footprint (none) -> flem:1Pin_d1.8mm_D3.4mm
- R101, R102: footprint Resistors_ThroughHole:Resistor_Horizontal_RM10mm -> Resistors_SMD:R_1206
- R103: renamed from R105; footprint Resistors_ThroughHole:Resistor_Horizontal_RM10mm -> Resistors_SMD:R_1206
- R104: renamed from R106; footprint Resistors_ThroughHole:Resistor_Horizontal_RM10mm -> Resistors_SMD:R_1206
- R105: renamed from R107; footprint Resistors_ThroughHole:Resistor_Horizontal_RM10mm -> Resistors_SMD:R_1206
- R106: renamed from R108; footprint Resistors_ThroughHole:Resistor_Horizontal_RM10mm -> Resistors_SMD:R_1206
- R107: renamed from R109; footprint Resistors_ThroughHole:Resistor_Horizontal_RM10mm -> Resistors_SMD:R_1206
- R108: renamed from R110; footprint Resistors_ThroughHole:Resistor_Horizontal_RM10mm -> Resistors_SMD:R_1206
- R109: renamed from R111; footprint Resistors_ThroughHole:Resistor_Horizontal_RM10mm -> Resistors_SMD:R_1206
- R110: renamed from R112; footprint Resistors_ThroughHole:Resistor_Horizontal_RM10mm -> Resistors_SMD:R_1206
Connections:
- net HP_Phone is gone; now on net S1: D101.2 (A)
- net +5V: now also K101.1 (+), K102.1 (+), K103.1 (+), K104.1 (+), K105.1 (+), K106.1 (+), P105.1 (P1)
- net GND: now also J114.2 (S), J112.2 (S)
- net PRE_IN_L: now also K101.4 (S), K102.4 (S), K103.4 (S), K104.4 (S), K105.4 (S)
- net PRE_IN_R: now also K101.5 (S), K102.5 (S), K103.5 (S), K104.5 (S), K105.5 (S)
- net PRE_OUT_L: now also K106.2 (O)
- net PRE_OUT_R: now also K106.7 (O)
- net S1: now also K101.8 (-), P105.2 (P2); no longer D102.2 (A)
- net S2: now also D102.2 (A), K102.8 (-), P105.3 (P3); no longer D103.2 (A)
- net S3: now also D103.2 (A), K103.8 (-), P105.4 (P4); no longer D104.2 (A)
- net S4: now also D104.2 (A), K104.8 (-), P105.5 (P5); no longer D105.2 (A)
- net S5: now also D105.2 (A), K105.8 (-), P105.6 (P6); no longer D106.2 (A)
- net at J101.1 (T), R101.1: now also K101.3 (P)
- net at J101.2 (S), J103.2 (S), J105.2 (S)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: now also R103.2; no longer R103.1
- net at J103.1 (T): now also R103.1, K102.3 (P); no longer R103.2
- net at J105.1 (T), R105.1: now also K103.3 (P)
- net at J107.1 (T), R107.1: now also K104.3 (P)
- net at J109.1 (T), R109.1: now also K105.3 (P)
- net at J102.1 (T), R102.1: now also K101.6 (P)
- net at J102.2 (S), J104.2 (S), J106.2 (S)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: no longer J114.2 (S)
- net at J104.1 (T), R104.1: now also K102.6 (P)
- net at J106.1 (T), R106.1: now also K103.6 (P)
- net at J108.1 (T), R108.1: now also K104.6 (P)
- net at J110.1 (T), R110.1: now also K105.6 (P)
- net at J114.1 (T): now also K106.5 (S)
- net at J111.1 (T): now also K106.3 (P)
- net at J113.1 (T): now also K106.6 (P)
- new net: J112.1 (T), K106.4 (S)
- new net BP: D106.2 (A), K106.8 (-), P105.7 (P7)
- no-connect marks 15 -> 10
Other:
- moved on the sheet: J111, J113, PA103, PA104, PB103, PB104
