File: KiCad/select_board/select_board.kicad_pcb (KiCad board)
At the start: 2 copper layers, 145.4 x 47.6 mm, 45 parts, among them J101 RCA, J102 RCA, J103 RCA, J104 RCA, J105 RCA, J106 RCA, J107 RCA, J108 RCA, J109 RCA, J110 RCA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

Commit message: Divers
Parts:
- moved P105 3.81 mm to (118.7, 103.5)
Routing:
- net +5V: track 132.1 -> 136.3 mm
- net GND: track 238.1 -> 241.8 mm
- net /S2: track 86.7 -> 88.3 mm
- net /S1: track 108.1 -> 109.7 mm
- net /BP: track 11.4 -> 9.78 mm
- net /S5: track 25.7 -> 24.2 mm
- net /S3: track 65.3 -> 66.9 mm

Commit message: Divers
Parts:
- moved K101 0.64 mm to (215.9, 111.1)
- moved K102 0.64 mm to (195.6, 111.1)
- moved K106 0.64 mm to (109.9, 111.1)
- moved K103 0.63 mm to (175.3, 111.1)
- moved K104 0.63 mm to (154.9, 111.1)
- moved K105 0.63 mm to (134.6, 111.1)
Routing:
- net +5V: track 136.3 -> 132.5 mm
- net /S2: track 88.3 -> 87.7 mm
- net /S1: track 109.7 -> 109.0 mm
- net /BP: track 9.78 -> 9.15 mm
- net /S5: track 24.2 -> 23.5 mm
- net /S4: track 45.5 -> 44.9 mm
- net /S3: track 66.9 -> 66.3 mm
- net /PRE_IN_L: track 107.6 -> 107.0 mm
- net /PRE_IN_R: track 107.7 -> 107.1 mm
- net Net-(J111-Pad1): track 39.9 -> 39.4 mm
