File: KiCad/mcu_board/mcu_board.kicad_pcb (KiCad board)
At the start: 2 copper layers, 99.1 x 69.8 mm, 24 parts, among them IC1 ATMEGA328P-AU, IC2 74HC595D, P1 CONN_02X04, P2 ICSP, P3 CONN_01X06, P4 CONN_01X02, P5 CONN_01X03, P6 CONN_01X04, P7 CONN_01X10, U1 ESP-02, U2 ULN2803A, U3 ULN2803A, U4 TSOP38238

Commit message: Gerber
Parts:
- removed the REF** at (76.2, 101.6)
- removed the REF** at (165.1, 101.6)
- added C101: 4.7uF, Capacitors_ThroughHole:CP_Radial_D5.0mm_P2.50mm, F.Cu at (113.0, 100.3)
- added R101: 150, Resistors_SMD:R_1206_HandSoldering, F.Cu at (111.8, 95.2)
- added REF**: MountingHole_3.2mm_M3_Pad, Mounting_Holes:MountingHole_3.2mm_M3_Pad, F.Cu at (165.1, 108.0)
- added REF**: MountingHole_3.2mm_M3_Pad, Mounting_Holes:MountingHole_3.2mm_M3_Pad, F.Cu at (76.2, 108.0)
Connections:
- U4 pad 3: +5P -> Net-(C101-Pad1)
Routing:
- net +3V3: track 95.3 -> 124.2 mm
- net Net-(C101-Pad1): track 0.00 -> 14.0 mm
- net GND: track 267.4 -> 259.1 mm, vias 10 -> 11
- net /LED_DIN: track 59.9 -> 65.7 mm
- net +5P: track 145.3 -> 143.4 mm

Commit message: Correctifs divers
Parts:
- U1: footprint franck:ESP_02_SMD_Handsoldering -> flem:ESP8266_ESP_02_SMD_Handsoldering
- U4: footprint franck:TSOP382 -> flem:TSOP382
- moved U1 13.6 mm to (142.9, 55.9), turned to 0 degrees
- moved P1 1.27 mm to (141.0, 71.1)
- moved REF** 0.90 mm to (164.5, 107.3)
Connections:
- P1 pad 3: /ESP-RX -> /ESP-TX
- P1 pad 5: /ESP-TX -> /ESP-RX
Routing:
- net GND: track 259.1 -> 289.9 mm, vias 11 -> 12
- net /ESP-GPIO2: track 28.6 -> 51.1 mm, vias 0 -> 1
- net /ESP-RST: track 10.6 -> 29.7 mm
- net /ESP-TX: track 86.6 -> 69.5 mm, vias 1 -> 2
- net /ESP-VCC: track 51.0 -> 39.4 mm, vias 2 -> 1
- net /ESP-GPIO15: track 22.5 -> 17.7 mm
- net /ESP-GPIO0: track 19.6 -> 21.5 mm
- net /LED_GND: track 57.4 -> 55.6 mm
- net /ESP-RX: track 79.1 -> 78.4 mm, vias 1 -> 2

Commit message: Gerber
Parts:
- removed U1: ESP-02, flem:ESP8266_ESP_02_SMD_Handsoldering
- added P106: CONN_01X02, Pin_Headers:Pin_Header_Straight_1x02_Pitch2.54mm, F.Cu at (165.1, 66.0)
- added U101: ESP-02, flem:ESP8266_ESP_02_SMD_Handsoldering, F.Cu at (142.9, 55.9)
- moved REF** 6.48 mm to (74.9, 101.6)
- moved REF** 6.02 mm to (166.4, 101.6)
- moved JP102 3.81 mm to (134.6, 47.0)
- moved C104 2.84 mm to (111.8, 102.9)
- moved U104 2.84 mm to (106.7, 110.5)
- moved P108 2.54 mm to (165.1, 71.1)
- moved JP101 2.54 mm to (132.1, 50.8)
- moved P107 2.54 mm to (165.1, 55.9)
- moved R101 1.91 mm to (154.9, 69.2)
- moved R102 1.91 mm to (158.8, 69.2)
- moved REF** 1.27 mm to (166.4, 48.3)
- moved REF** 1.27 mm to (74.9, 48.3)
- moved R103 0.64 mm to (111.8, 95.9), turned to 90 degrees
- renumbered C3 to C101, C4 to C102, C1 to C103, C101 to C104, IC1 to IC101, IC2 to IC102, JP1 to JP101, JP2 to JP102, P1 to P101, P2 to P102, P3 to P103, P4 to P104, P5 to P105, P6 to P107, P7 to P108, R1 to R101, R2 to R102, R101 to R103, U2 to U102, U3 to U103, U4 to U104
Connections:
- IC101 pad 10: (no net) -> /FU2
- IC101 pad 11: (no net) -> Net-(IC101-Pad11)
- IC101 pad 13: (no net) -> Net-(IC101-Pad13)
- IC101 pad 19: (no net) -> Net-(IC101-Pad19)
- IC101 pad 2: (no net) -> Net-(IC101-Pad2)
- IC101 pad 20: (no net) -> Net-(IC101-Pad20)
- IC101 pad 22: (no net) -> Net-(IC101-Pad22)
- IC101 pad 7: (no net) -> Net-(IC101-Pad7)
- IC101 pad 8: (no net) -> Net-(IC101-Pad8)
- IC101 pad 9: (no net) -> /FU1
- IC102 pad 9: (no net) -> Net-(IC102-Pad9)
- JP102 pad 1: /ESP-GPIO2 -> /ESP-RST
- P101 pad 8: /ESP-GPIO15 -> /ESP-CHPD
- P108 pad 10: (no net) -> Net-(P108-Pad10)
- U102 pad 10: (no net) -> Net-(U102-Pad10)
- U103 pad 10: (no net) -> Net-(U103-Pad10)
- U103 pad 11: (no net) -> Net-(U103-Pad11)
- U103 pad 12: (no net) -> Net-(U103-Pad12)
- U103 pad 13: (no net) -> Net-(U103-Pad13)
- U103 pad 14: (no net) -> /K-FU2
- U103 pad 15: (no net) -> /K-FU1
- U103 pad 4: (no net) -> /FU1
- U103 pad 5: (no net) -> /FU2
- U103 pad 6: (no net) -> Net-(U103-Pad6)
- U103 pad 7: (no net) -> Net-(U103-Pad7)
- U103 pad 8: (no net) -> Net-(U103-Pad8)
Routing:
- net GND: track 289.9 -> 53.3 mm, vias 12 -> 2
- net +5P: track 143.4 -> 89.8 mm
- net /K-FU1: track 0.00 -> 44.6 mm, vias 0 -> 1
- net /K-FU2: track 0.00 -> 44.5 mm, vias 0 -> 1
- net /FU1: track 0.00 -> 23.9 mm, vias 0 -> 2
- net /ESP-GPIO2: track 51.1 -> 27.7 mm, vias 1 -> 0
- net /FU2: track 0.00 -> 22.2 mm, vias 0 -> 2
- net /ESP-RST: track 29.7 -> 48.6 mm
- net /ESP-GPIO15: track 17.7 -> 0.00 mm
- net /ESP-CHPD: track 0.00 -> 17.7 mm
- net /RESET: track 72.5 -> 85.5 mm, vias 2 -> 3
- net /s1: track 44.1 -> 38.4 mm
- net /LED_DIN: track 65.7 -> 60.1 mm
- net /LED_GND: track 55.6 -> 50.7 mm
- net /SCL: track 80.3 -> 83.8 mm
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Other:
- board size 99.1 x 69.8 mm -> 99.1 x 68.6 mm

Commit message: Divers
Connections:
- JP102 pad 1: /ESP-RST -> /ESP-GPIO2
Routing:
- net /ESP-GPIO2: track 27.7 -> 58.5 mm
- net /ESP-RST: track 48.6 -> 31.3 mm

Commit message: Divers
Connections:
- net /hp renamed /s8
- IC101 pad 11: Net-(IC101-Pad11) -> (no net)
- IC101 pad 13: Net-(IC101-Pad13) -> (no net)
- IC101 pad 19: Net-(IC101-Pad19) -> (no net)
- IC101 pad 2: Net-(IC101-Pad2) -> (no net)
- IC101 pad 20: Net-(IC101-Pad20) -> (no net)
- IC101 pad 22: Net-(IC101-Pad22) -> (no net)
- IC101 pad 7: Net-(IC101-Pad7) -> (no net)
- IC101 pad 8: Net-(IC101-Pad8) -> (no net)
- IC102 pad 9: Net-(IC102-Pad9) -> (no net)
- P108 pad 10: Net-(P108-Pad10) -> (no net)
- U102 pad 10: Net-(U102-Pad10) -> (no net)
- U103 pad 10: Net-(U103-Pad10) -> (no net)
- U103 pad 11: Net-(U103-Pad11) -> (no net)
- U103 pad 12: Net-(U103-Pad12) -> (no net)
- U103 pad 13: Net-(U103-Pad13) -> (no net)
- U103 pad 6: Net-(U103-Pad6) -> (no net)
- U103 pad 7: Net-(U103-Pad7) -> (no net)
- U103 pad 8: Net-(U103-Pad8) -> (no net)
